Commit message: Changing axis...

File: lab2/urdf/dynamic.urdf (robot description, URDF)
Before this commit: robot example_robot, 4 links, 3 joints
Joints:
- joint link1_to_link2: axis 0 0 1 -> 1 0 0

Commit message: small visual upgrade

File: lab2/urdf/dynamic.urdf (robot description, URDF)
Before this commit: robot example_robot, 4 links, 3 joints
Links:
- link link_1: geometry visual box size=${l_width} 1.0 ${l_width}
- link link_2: geometry visual box size=${l_width} 2.0 ${l_width}
Joints:
- joint link1_to_link2: limit lower=-1.57075 upper=1.57075 effort=1000.0 velocity=0.5 -> lower=1.57075 upper=0 effort=1000.0 velocity=0.5

File: lab2/urdf/static.urdf (robot description, URDF)
Before this commit: robot example_robot, 4 links, 3 joints
Links:
- link link_1: geometry visual box size=${l_width} 1.0 ${l_width}
- link link_2: geometry visual box size=${l_width} 2.0 ${l_width}

Commit message: Replanning projekt 2 and start of 3

File: lab2/urdf/dynamic.urdf (robot description, URDF)
Before this commit: robot example_robot, 4 links, 3 joints
Links:
- link link_1: geometry visual box size=${l_width} ${l_width} ${props['i2']['l_len']}
- link link_2: geometry visual box size=${l_width} ${l_width} ${props['i3']['l_len']}
- link link_3: geometry visual box size=${l_width} ${l_width} 2; visual mesh filename=package://lab2/FuturamaRifle.stl scale=0.001 0.001 0.002
Joints:
- joint base_to_link1: limit lower=-1.57075 upper=1.57075 effort=1000.0 velocity=0.5 -> lower=-${props['i2']['l_len']} upper=0 effort=1000.0 velocity=0.5; type revolute -> prismatic
- joint link1_to_link2: axis 1 0 0 -> 0 0 1; limit lower=1.57075 upper=0 effort=1000.0 velocity=0.5 -> lower=-${props['i3']['l_len']} upper=0 effort=1000.0 velocity=0.5; type revolute -> prismatic
- joint link2_to_link3: limit lower=-1.57075 upper=1.57075 effort=1000.0 velocity=0.5 -> lower=-1 upper=1 effort=1000.0 velocity=0.5; type revolute -> prismatic

File: lab2/urdf/static.urdf (robot description, URDF)
Before this commit: robot example_robot, 4 links, 3 joints
Links:
- link link_1: geometry visual box size=${l_width} ${l_width} ${props['i2']['l_len']}
- link link_2: geometry visual box size=${l_width} ${l_width} ${props['i3']['l_len']}
- link link_3: geometry visual box size=${l_width} ${l_width} 2; visual mesh filename=package://lab2/FuturamaRifle.stl scale=0.001 0.001 0.002
