Commit message: Final dynamic

File: lab2/urdf/static.urdf (robot description, URDF)
Before this commit: robot example_robot, 14 links, 13 joints
Links:
- removed link link0_passive
- removed link link0_x_axis
- removed link link1
- removed link link1_passive
- removed link link1_x_axis
- removed link link2
- removed link link2_passive
- removed link link2_x_axis
- removed link link3
- removed link link3_passive
- removed link link3_x_axis
- removed link link4
- removed link link4_passive
- removed link link4_x_axis
- added link base_link; visual cylinder length=0.04 radius=0.05
- added link link_1; visual box size=${props['i2']['l_len']} ${l_width} ${l_width}
- added link link_2; visual box size=${props['i3']['l_len']} ${l_width} ${l_width}
- added link link_3; visual mesh filename=package://lab2/hand.stl scale=0.001 0.001 0.002
Joints:
- removed joint q0_x
- removed joint q1
- removed joint q1_passive
- removed joint q1_x
- removed joint q2
- removed joint q2_passive
- removed joint q2_x
- removed joint q3
- removed joint q3_passive
- removed joint q3_x
- removed joint q4
- removed joint q4_passive
- removed joint q4_x
- added joint base_to_link1: type revolute, parent base_link, child link_1, origin xyz=${props['i1']['j_xyz']} rpy=${props['i1']['j_rpy']}, axis 0 0 1, limit lower=-1.57075 upper=1.57075 effort=1000.0 velocity=0.5
- added joint link1_to_link2: type revolute, parent link_1, child link_2, origin xyz=${props['i2']['j_xyz']} rpy=${props['i2']['j_rpy']}, axis 0 0 1, limit lower=-1.57075 upper=1.57075 effort=1000.0 velocity=0.5
- added joint link2_to_link3: type prismatic, parent link_2, child link_3, origin xyz=${props['i3']['j_xyz']} rpy=${props['i3']['j_rpy']}, axis 0 0 1, limit lower=0 upper=0.2 effort=1000.0 velocity=0.5

Commit message: Static & Dynamic fin

File: lab2/urdf/static.urdf (robot description, URDF)
Before this commit: robot example_robot, 4 links, 3 joints
Links:
- link link_3: geometry visual mesh filename=package://lab2/FuturamaRifle.stl scale=0.001 0.001 0.002
Joints:
- joint base_to_link1: axis 0 0 1 -> (none); limit lower=-1.57075 upper=1.57075 effort=1000.0 velocity=0.5 -> (none); type revolute -> fixed
- joint link1_to_link2: axis 0 0 1 -> (none); limit lower=-1.57075 upper=1.57075 effort=1000.0 velocity=0.5 -> (none); type revolute -> fixed
- joint link2_to_link3: axis 0 0 1 -> (none); limit lower=0 upper=0.2 effort=1000.0 velocity=0.5 -> (none); type prismatic -> fixed

Commit message: Final version

File: lab2/urdf/static.urdf (robot description, URDF)
Before this commit: robot example_robot, 4 links, 3 joints
Links:
- link link_1: geometry visual box size=${l_width} ${l_width} ${props['i1']['l_len']}
- link link_2: geometry visual box size=${l_width} ${l_width} ${props['i2']['l_len']}
- link link_3: geometry visual box size=${l_width} ${l_width} ${props['i3']['l_len']}; visual mesh filename=package://lab2/FuturamaRifle.stl scale=0.001 0.001 0.002

File: lab2/urdf/test.urdf (robot description, URDF)
Before this commit: robot example_robot, 4 links, 3 joints
Links:
- link link_1: geometry visual box size=0.02 0.02 1
- link link_2: geometry visual box size=0.02 0.02 1
- link link_3: geometry visual box size=0.02 0.02 1; visual mesh filename=package://lab2/FuturamaRifle.stl scale=0.001 0.001 0.002
Joints:
- joint base_to_link1: limit lower=-${props['i1']['l_len']} upper=0 effort=1000.0 velocity=0.5 -> lower=-1 upper=0 effort=1000.0 velocity=0.5; origin xyz=${props['i1']['j_xyz']} rpy=${props['i1']['j_rpy']} -> xyz=0 0 1 rpy=0 0 0
- joint link1_to_link2: limit lower=-${props['i2']['l_len']} upper=0 effort=1000.0 velocity=0.5 -> lower=-1 upper=0 effort=1000.0 velocity=0.5; origin xyz=${props['i2']['j_xyz']} rpy=${props['i2']['j_rpy']} -> xyz=0 -1 0 rpy=1.57075 -1.57075 0
- joint link2_to_link3: limit lower=-${props['i3']['l_len']} upper=0 effort=1000.0 velocity=0.5 -> lower=-1 upper=0 effort=1000.0 velocity=0.5; origin xyz=${props['i3']['j_xyz']} rpy=${props['i3']['j_rpy']} -> xyz=0 -1 0 rpy=1.57075 -1.57075 0
